File: lboard.sch (KiCad schematic (older format))
At the start: 24 parts, among them P1 CONN_01X02_PWR, U1 AP1117_ADJ, U2 AP1117_33, U3 AP1117_ADJ

Commit message: footprint of oscillator Y1 changed. Some silscreen changes
Parts:
- GNDTST1: symbol TEST -> TEST-RESCUE-lboard
Changed lines of the file:
@@
 EESchema Schematic File Version 2
+LIBS:lboard-rescue
 LIBS:power
 LIBS:device
@@
 CD[0..7]
 $Comp
-L TEST GNDTST1
+L TEST-RESCUE-lboard GNDTST1
 U 1 1 584A94E7
 P 3875 2525
